File: schematics/untitled.kicad_sch (KiCad schematic)
At the start: 150 parts, among them SW1 SW_Push, SW10 SW_Push, SW11 SW_Push, SW12 SW_Push, SW13 SW_Push, SW14 SW_Push, SW15 SW_Push, SW16 SW_Push, SW17 SW_Push, SW18 SW_Push, SW19 SW_Push, SW2 SW_Push, SW20 SW_Push, SW21 SW_Push, SW22 SW_Push, SW23 SW_Push, SW24 SW_Push, SW25 SW_Push, SW26 SW_Push, SW27 SW_Push, SW28 SW_Push, SW29 SW_Push, SW3 SW_Push, SW30 SW_Push, SW31 SW_Push, SW32 SW_Push, SW33 SW_Push, SW34 SW_Push, SW35 SW_Push, SW36 SW_Push, SW37 SW_Push, SW38 SW_Push, SW39 SW_Push, SW4 SW_Push, SW40 SW_Push, SW41 SW_Push, SW42 SW_Push, SW43 SW_Push, SW44 SW_Push, SW45 SW_Push, SW46 SW_Push, SW47 SW_Push, SW48 SW_Push, SW49 SW_Push, SW5 SW_Push, SW50 SW_Push, SW51 SW_Push, SW52 SW_Push, SW53 SW_Push, SW54 SW_Push, SW55 SW_Push, SW56 SW_Push, SW57 SW_Push, SW58 SW_Push, SW59 SW_Push, SW6 SW_Push, SW60 SW_Push, SW61 SW_Push, SW62 SW_Push, SW63 SW_Push, SW64 SW_Push, SW65 SW_Push, SW66 SW_Push, SW67 SW_Push, SW68 SW_Push, SW69 SW_Push, SW7 SW_Push, SW70 SW_Push, SW71 SW_Push, SW72 SW_Push, SW73 SW_Push, SW74 SW_Push, SW75 SW_Push, SW8 SW_Push, SW9 SW_Push

Commit message: (feat) add power flash usb and clock to sch
Parts:
- D1, D10, D11, D12, D13, D14, D15, D16, D17, D18, D19, D2, D20, D21, D22, D23, D24, D25, D26, D27, D28, D29, D3, D30, D31, D32, D33, D34, D35, D36, D37, D38, D39, D4, D40, D41, D42, D43, D44, D45, D46, D47, D48, D49, D5, D50, D51, D52, D53, D54, D55, D56, D57, D58, D59, D6, D60, D61, D62, D63, D64, D65, D66, D67, D68, D69, D7, D70, D71, D72, D73, D74, D75, D8, D9: footprint Diode_THT:D_DO-41_SOD81_P10.16mm_Horizontal -> Diode_SMD:D_0201_0603Metric

Commit message: (feat) first layout
Parts:
- removed D15, D28, D30, D43, D45, D60, D65, D66, D67, D69, D70, D75: 1N4002, Diode_SMD:D_0201_0603Metric, symbol Diode:1N4002
- removed SW15, SW28, SW30, SW43, SW45, SW60, SW65, SW66, SW67, SW69, SW70, SW75: SW_Push, symbol Switch:SW_Push
- added D27: 1N4002, Diode_SMD:D_SOD-123, symbol Diode:1N4002
- added S1: MX_stab, PCM_marbastlib-mx:STAB_MX_P_6u, symbol PCM_marbastlib-mx:MX_stab
- added SW27: SW_Push, PCM_marbastlib-mx:SW_MX_1u, symbol Switch:SW_Push
- D1, D10, D11, D12, D13, D14, D2, D3, D4, D5, D6, D7, D8, D9: footprint Diode_SMD:D_0201_0603Metric -> Diode_SMD:D_SOD-123
- D15: renamed from D16; footprint Diode_SMD:D_0201_0603Metric -> Diode_SMD:D_SOD-123
- D16: renamed from D17; footprint Diode_SMD:D_0201_0603Metric -> Diode_SMD:D_SOD-123
- D17: renamed from D18; footprint Diode_SMD:D_0201_0603Metric -> Diode_SMD:D_SOD-123
- D18: renamed from D19; footprint Diode_SMD:D_0201_0603Metric -> Diode_SMD:D_SOD-123
- D19: renamed from D20; footprint Diode_SMD:D_0201_0603Metric -> Diode_SMD:D_SOD-123
- D20: renamed from D21; footprint Diode_SMD:D_0201_0603Metric -> Diode_SMD:D_SOD-123
- D21: renamed from D22; footprint Diode_SMD:D_0201_0603Metric -> Diode_SMD:D_SOD-123
- D22: renamed from D23; footprint Diode_SMD:D_0201_0603Metric -> Diode_SMD:D_SOD-123
- D23: renamed from D24; footprint Diode_SMD:D_0201_0603Metric -> Diode_SMD:D_SOD-123
- D24: renamed from D25; footprint Diode_SMD:D_0201_0603Metric -> Diode_SMD:D_SOD-123
- D25: renamed from D26; footprint Diode_SMD:D_0201_0603Metric -> Diode_SMD:D_SOD-123
- D26: renamed from D27; footprint Diode_SMD:D_0201_0603Metric -> Diode_SMD:D_SOD-123
- D28: renamed from D29; footprint Diode_SMD:D_0201_0603Metric -> Diode_SMD:D_SOD-123
- D29: renamed from D31; footprint Diode_SMD:D_0201_0603Metric -> Diode_SMD:D_SOD-123
- D30: renamed from D32; footprint Diode_SMD:D_0201_0603Metric -> Diode_SMD:D_SOD-123
- D31: renamed from D33; footprint Diode_SMD:D_0201_0603Metric -> Diode_SMD:D_SOD-123
- D32: renamed from D34; footprint Diode_SMD:D_0201_0603Metric -> Diode_SMD:D_SOD-123
- D33: renamed from D35; footprint Diode_SMD:D_0201_0603Metric -> Diode_SMD:D_SOD-123
- D34: renamed from D36; footprint Diode_SMD:D_0201_0603Metric -> Diode_SMD:D_SOD-123
- D35: renamed from D37; footprint Diode_SMD:D_0201_0603Metric -> Diode_SMD:D_SOD-123
- D36: renamed from D38; footprint Diode_SMD:D_0201_0603Metric -> Diode_SMD:D_SOD-123
- D37: renamed from D39; footprint Diode_SMD:D_0201_0603Metric -> Diode_SMD:D_SOD-123
- D38: renamed from D40; footprint Diode_SMD:D_0201_0603Metric -> Diode_SMD:D_SOD-123
- D39: renamed from D41; footprint Diode_SMD:D_0201_0603Metric -> Diode_SMD:D_SOD-123
- D40: renamed from D42; footprint Diode_SMD:D_0201_0603Metric -> Diode_SMD:D_SOD-123
- D41: renamed from D44; footprint Diode_SMD:D_0201_0603Metric -> Diode_SMD:D_SOD-123
- D42: renamed from D46; footprint Diode_SMD:D_0201_0603Metric -> Diode_SMD:D_SOD-123
- D43: renamed from D47; footprint Diode_SMD:D_0201_0603Metric -> Diode_SMD:D_SOD-123
- D44: renamed from D48; footprint Diode_SMD:D_0201_0603Metric -> Diode_SMD:D_SOD-123
- D45: renamed from D49; footprint Diode_SMD:D_0201_0603Metric -> Diode_SMD:D_SOD-123
- D46: renamed from D50; footprint Diode_SMD:D_0201_0603Metric -> Diode_SMD:D_SOD-123
- D47: renamed from D51; footprint Diode_SMD:D_0201_0603Metric -> Diode_SMD:D_SOD-123
- D48: renamed from D52; footprint Diode_SMD:D_0201_0603Metric -> Diode_SMD:D_SOD-123
- D49: renamed from D53; footprint Diode_SMD:D_0201_0603Metric -> Diode_SMD:D_SOD-123
- D50: renamed from D54; footprint Diode_SMD:D_0201_0603Metric -> Diode_SMD:D_SOD-123
- D51: renamed from D55; footprint Diode_SMD:D_0201_0603Metric -> Diode_SMD:D_SOD-123
- D52: renamed from D56; footprint Diode_SMD:D_0201_0603Metric -> Diode_SMD:D_SOD-123
- D53: renamed from D57; footprint Diode_SMD:D_0201_0603Metric -> Diode_SMD:D_SOD-123
- D54: renamed from D58; footprint Diode_SMD:D_0201_0603Metric -> Diode_SMD:D_SOD-123
- D55: renamed from D59; footprint Diode_SMD:D_0201_0603Metric -> Diode_SMD:D_SOD-123
- D56: renamed from D61; footprint Diode_SMD:D_0201_0603Metric -> Diode_SMD:D_SOD-123
- D57: renamed from D62; footprint Diode_SMD:D_0201_0603Metric -> Diode_SMD:D_SOD-123
- D58: renamed from D63; footprint Diode_SMD:D_0201_0603Metric -> Diode_SMD:D_SOD-123
- D59: renamed from D64; footprint Diode_SMD:D_0201_0603Metric -> Diode_SMD:D_SOD-123
- D60: renamed from D68; footprint Diode_SMD:D_0201_0603Metric -> Diode_SMD:D_SOD-123
- D61: renamed from D71; footprint Diode_SMD:D_0201_0603Metric -> Diode_SMD:D_SOD-123
- D62: renamed from D72; footprint Diode_SMD:D_0201_0603Metric -> Diode_SMD:D_SOD-123
- D63: renamed from D73; footprint Diode_SMD:D_0201_0603Metric -> Diode_SMD:D_SOD-123
- D64: renamed from D74; footprint Diode_SMD:D_0201_0603Metric -> Diode_SMD:D_SOD-123
- SW1, SW10, SW11, SW12, SW13, SW2, SW3, SW4, SW5, SW6, SW7, SW8, SW9: footprint (none) -> PCM_marbastlib-mx:SW_MX_1u
- SW14: footprint (none) -> PCM_marbastlib-mx:SW_MX_1.5u
- SW15: renamed from SW16; footprint (none) -> PCM_marbastlib-mx:SW_MX_1.5u
- SW16: renamed from SW17; footprint (none) -> PCM_marbastlib-mx:SW_MX_1u
- SW17: renamed from SW18; footprint (none) -> PCM_marbastlib-mx:SW_MX_1u
- SW18: renamed from SW19; footprint (none) -> PCM_marbastlib-mx:SW_MX_1u
- SW19: renamed from SW20; footprint (none) -> PCM_marbastlib-mx:SW_MX_1u
- SW20: renamed from SW21; footprint (none) -> PCM_marbastlib-mx:SW_MX_1u
- SW21: renamed from SW22; footprint (none) -> PCM_marbastlib-mx:SW_MX_1u
- SW22: renamed from SW23; footprint (none) -> PCM_marbastlib-mx:SW_MX_1u
- SW23: renamed from SW24; footprint (none) -> PCM_marbastlib-mx:SW_MX_1u
- SW24: renamed from SW25; footprint (none) -> PCM_marbastlib-mx:SW_MX_1u
- SW25: renamed from SW26; footprint (none) -> PCM_marbastlib-mx:SW_MX_1u
- SW26: renamed from SW27; footprint (none) -> PCM_marbastlib-mx:SW_MX_1u
- SW28: renamed from SW29; footprint (none) -> PCM_marbastlib-mx:SW_MX_1u
- SW29: renamed from SW31; footprint (none) -> PCM_marbastlib-mx:SW_MX_1.75u
- SW30: renamed from SW32; footprint (none) -> PCM_marbastlib-mx:SW_MX_1u
- SW31: renamed from SW33; footprint (none) -> PCM_marbastlib-mx:SW_MX_1u
- SW32: renamed from SW34; footprint (none) -> PCM_marbastlib-mx:SW_MX_1u
- SW33: renamed from SW35; footprint (none) -> PCM_marbastlib-mx:SW_MX_1u
- SW34: renamed from SW36; footprint (none) -> PCM_marbastlib-mx:SW_MX_1u
- SW35: renamed from SW37; footprint (none) -> PCM_marbastlib-mx:SW_MX_1u
- SW36: renamed from SW38; footprint (none) -> PCM_marbastlib-mx:SW_MX_1u
- SW37: renamed from SW39; footprint (none) -> PCM_marbastlib-mx:SW_MX_1u
- SW38: renamed from SW40; footprint (none) -> PCM_marbastlib-mx:SW_MX_1u
- SW39: renamed from SW41; footprint (none) -> PCM_marbastlib-mx:SW_MX_1u
- SW40: renamed from SW42; footprint (none) -> PCM_marbastlib-mx:SW_MX_1u
- SW41: renamed from SW44; footprint (none) -> PCM_marbastlib-mx:SW_MX_1.75u
- SW42: renamed from SW46; footprint (none) -> PCM_marbastlib-mx:SW_MX_1.5u
- SW43: renamed from SW47; footprint (none) -> PCM_marbastlib-mx:SW_MX_1u
- SW44: renamed from SW48; footprint (none) -> PCM_marbastlib-mx:SW_MX_1u
- SW45: renamed from SW49; footprint (none) -> PCM_marbastlib-mx:SW_MX_1u
- SW46: renamed from SW50; footprint (none) -> PCM_marbastlib-mx:SW_MX_1u
- SW47: renamed from SW51; footprint (none) -> PCM_marbastlib-mx:SW_MX_1u
- SW48: renamed from SW52; footprint (none) -> PCM_marbastlib-mx:SW_MX_1u
- SW49: renamed from SW53; footprint (none) -> PCM_marbastlib-mx:SW_MX_1u
- SW50: renamed from SW54; footprint (none) -> PCM_marbastlib-mx:SW_MX_1u
- SW51: renamed from SW55; footprint (none) -> PCM_marbastlib-mx:SW_MX_1u
- SW52: renamed from SW56; footprint (none) -> PCM_marbastlib-mx:SW_MX_1u
- SW53: renamed from SW57; footprint (none) -> PCM_marbastlib-mx:SW_MX_1u
- SW54: renamed from SW58; footprint (none) -> PCM_marbastlib-mx:SW_MX_1u
- SW55: renamed from SW59; footprint (none) -> PCM_marbastlib-mx:SW_MX_1u
- SW56: renamed from SW61; footprint (none) -> PCM_marbastlib-mx:SW_MX_1.25u
- SW57: renamed from SW62; footprint (none) -> PCM_marbastlib-mx:SW_MX_1u
- SW58: renamed from SW63; footprint (none) -> PCM_marbastlib-mx:SW_MX_1u
- SW59: renamed from SW64; footprint (none) -> PCM_marbastlib-mx:SW_MX_1u
- SW60: renamed from SW68; footprint (none) -> PCM_marbastlib-mx:SW_MX_1u
- SW61: renamed from SW71; footprint (none) -> PCM_marbastlib-mx:SW_MX_1.25u
- SW62: renamed from SW72; footprint (none) -> PCM_marbastlib-mx:SW_MX_1u
- SW63: renamed from SW73; footprint (none) -> PCM_marbastlib-mx:SW_MX_1u
- SW64: renamed from SW74; footprint (none) -> PCM_marbastlib-mx:SW_MX_1u
Connections:
- net Col12: now also SW27.2
- net Row1: now also D27.2 (A)
- new net: D27.1 (K), SW27.1
